File: Winkdings2.kicad_pcb (KiCad board)
At the start: 2 copper layers, 59.4 x 76.2 mm, 20 parts, among them SW1 TS665CJ, U1 FabCore2_Module

Commit message: fixed gnd plane
Routing:
- added copper zone on B.Cu, net GND
- added copper zone on F.Cu, net GND
Changed lines of the file:
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@@
 		(net "Net-(D5-K)")
+	)
+	(zone
+		(net "GND")
+		(layers "F.Cu" "B.Cu")
+		(hatch edge 0.5)
+		(connect_pads
+			(clearance 0.5)
+		)
+		(min_thickness 0.25)
+		(fill yes
+			(thermal_gap 0.5)
+			(thermal_bridge_width 0.5)
+			(smoothing chamfer)
+			(radius 1)
+			(island_removal_mode 0)
+		)
+		(polygon
+			(pts
+				(xy 104.394 51.562) (xy 171.958 51.562) (xy 171.704 137.922) (xy 105.664 137.414)
+			)
+		)
 	)
 	(embedded_fonts no)
